File: Reciver/HW/V1/main/main.sch (KiCad schematic (older format))
At the start: 13 parts, among them U1 NodeMCU_1.0_(ESP-12E), U2 RFM95W-868S2, U3 NodeMCU_1.0_(ESP-12E)

Commit message: layout
kicad
Parts:
- removed MH1, MH2, MH3, MH4: MountingHole, MountingHole:MountingHole_3.2mm_M3, symbol Mechanical:MountingHole
- removed U3: NodeMCU_1.0_(ESP-12E), ESP8266:NodeMCU1.0(12-E), symbol ESP8266:NodeMCU_1.0_(ESP-12E)
Changed lines of the file:
@@
 Wire Wire Line
 	4750 2600 4300 2600
-$Comp
-L Mechanical:MountingHole MH2
-U 1 1 5B6728D5
-P 4350 4900
-F 0 "MH2" H 4450 4946 50  0000 L CNN
-F 1 "MountingHole" H 4450 4855 50  0000 L CNN
-F 2 "MountingHole:MountingHole_3.2mm_M3" H 4350 4900 50  0001 C CNN
-F 3 "~" H 4350 4900 50  0001 C CNN
-	1    4350 4900
-	1    0    0    -1
-$EndComp
-$Comp
-L Mechanical:MountingHole MH3
-U 1 1 5B672909
-P 5100 4900
-F 0 "MH3" H 5200 4946 50  0000 L CNN
-F 1 "MountingHole" H 5200 4855 50  0000 L CNN
-F 2 "MountingHole:MountingHole_3.2mm_M3" H 5100 4900 50  0001 C CNN
-F 3 "~" H 5100 4900 50  0001 C CNN
-	1    5100 4900
-	1    0    0    -1
-$EndComp
-$Comp
-L Mechanical:MountingHole MH4
-U 1 1 5B672947
-P 5150 5350
-F 0 "MH4" H 5250 5396 50  0000 L CNN
-F 1 "MountingHole" H 5250 5305 50  0000 L CNN
-F 2 "MountingHole:MountingHole_3.2mm_M3" H 5150 5350 50  0001 C CNN
-F 3 "~" H 5150 5350 50  0001 C CNN
-	1    5150 5350
-	1    0    0    -1
-$EndComp
-$Comp
-L Mechanical:MountingHole MH1
-U 1 1 5B672981
-P 4300 5350
-F 0 "MH1" H 4400 5396 50  0000 L CNN
-F 1 "MountingHole" H 4400 5305 50  0000 L CNN
-F 2 "MountingHole:MountingHole_3.2mm_M3" H 4300 5350 50  0001 C CNN
-F 3 "~" H 4300 5350 50  0001 C CNN
-	1    4300 5350
-	1    0    0    -1
-$EndComp
-$Comp
-L ESP8266:NodeMCU_1.0_(ESP-12E) U3
-U 1 1 5B674F2D
-P 6550 1600
-F 0 "U3" H 6550 2687 60  0000 C CNN
-F 1 "NodeMCU_1.0_(ESP-12E)" H 6550 2581 60  0000 C CNN
-F 2 "ESP8266:NodeMCU1.0(12-E)" H 5950 750 60  0001 C CNN
-F 3 "" H 5950 750 60  0000 C CNN
-	1    6550 1600
-	1    0    0    -1
-$EndComp
 $EndSCHEMATC
