File: MountedOnMailbox/HW/V2/main.sch (KiCad schematic (older format))
At the start: 34 parts, among them J1 BoxLidSensor, J2 CONSMA001-SMD-G, J3 FTDI, J4 AVR-ISP-6, Q1 IRF7341, SW1 Reset, U1 ATMEGA328P-AU-Arduino, U2 RFM95W-868S2, U3 DW01-P, U4 AP2210-3.3V, Y1 8MHz

Commit message: Better layout
And i2c header
Parts:
- added C13: 100n, Capacitor_SMD:C_0805_2012Metric_Pad1.15x1.40mm_HandSolder, symbol Device:C
- added J5: Conn_01x04_Female, Connector_PinHeader_2.54mm:PinHeader_1x04_P2.54mm_Vertical, symbol Connector:Conn_01x04_Female
- C1: value C -> 100n
- J2: footprint Connector_Coaxial:SMA_Molex_73251-1153_EdgeMount_Horizontal -> Libs:SMA_edge connector
- TP1: symbol Connector:Test_Point -> main-rescue:Test_Point-Connector
Connections:
- net labels added: SCL, SDA
- net labels removed: scl, sda
- wire segments 110 -> 108
Other:
- note added: "I2C Header"
- note removed: "Reset\n"
- moved on the sheet: C1, J1, R1, R2, SW1
